File: robot-cortex.kicad_pcb (KiCad board)
At the start: 4 copper layers, 27.5 x 35.8 mm, 91 parts, among them IC1 THVD2450VDRCR, IC2 THVD2450VDRCR, IC3 THVD2450VDRCR, J1 USB4110GFA, M1 THRU_HOLE_PAD, M2 THRU_HOLE_PAD, Q1 SSM3K15F,LF, Q2 SSM3K15F,LF, U1 C2901617, U10 TPS63070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

Commit message: Updated power distribution - now RS485 breaks out 7V, and the buckboost produces 7V. Battery input comes from the CAN connector alone. This way 1S lipo works, 2S lipo works, up to 16VDC input for VBAT, and USB can power the gate drivers for motors, elimintaing a power supply dependency or external buck converter for batteries in systems which use this as the primary processor
Parts:
- removed R16: 0, robot-cortex:R_0402_1005Metric
- added D9: ESD9B3.3ST5G, robot-cortex:D_SOD-923, B.Cu at (192.9, 113.2)
- R13: value 680k -> 365k
- R14: value 130k -> 47k
- moved C33 9.76 mm to (192.1, 105.4), turned to 180 degrees
- moved C32 2.31 mm to (196.3, 113.7), turned to -90 degrees
- moved C9 1.98 mm to (198.2, 112.5), turned to 0 degrees
- moved C24 1.33 mm to (196.1, 111.1)
Connections:
- C11 pad 1: /VBAT -> /7V0
- C12 pad 1: /VBAT -> /7V0
- C24 pad 1: /+5V0 -> /7V0
- C32 pad 1: /+5V0 -> /7V0
- C33 pad 1: /+5V0 -> /7V0
- D8 pad 2: /VBAT -> /7V0
- R13 pad 1: /+5V0 -> /7V0
- R15 pad 1: /+5V0 -> /7V0
- U11 pad 7,8: /+5V0 -> /7V0
- U12 pad 1: /VBAT -> /7V0
- U13 pad 1: /VBAT -> /7V0
- U14 pad 1: /VBAT -> /7V0
- U6 pad 1: /VBAT -> /7V0
- U6 pad 3: /VBAT -> /7V0
Routing:
- net /7V0: track 0.00 -> 58.4 mm, vias 0 -> 2
- net /VBAT: track 60.3 -> 8.95 mm, vias 1 -> 0
- net /+5V0: track 70.4 -> 58.6 mm
- net /VUSB: track 16.0 -> 14.0 mm, vias 3 -> 2
- net +3V3: track 53.9 -> 52.7 mm
- net /UART1_TX: track 11.3 -> 11.8 mm
- net GND: vias 96 -> 101
- added copper zone on F.Cu, net /7V0
- removed copper zone on F.Cu, net /+5V0
Other:
- board text added: "7V0 A B GND"
- board text removed: "Vbat A B GND"
