File: robot-cortex.kicad_sch (KiCad schematic)
At the start: 40 parts, among them J1 USB4110GFA, M1 THRU_HOLE_PAD, M2 THRU_HOLE_PAD, U1 C2901617, U2 STM32G431CBT6, U3 TLE9250XSJXUMA1, U4 DF52-3S-0.8H(21), U5 DF52-4S-0.8H(21), U6 SPX3819M5-L-5-0

Commit message: Updated power distribution - now RS485 breaks out 7V, and the buckboost produces 7V. Battery input comes from the CAN connector alone. This way 1S lipo works, 2S lipo works, up to 16VDC input for VBAT, and USB can power the gate drivers for motors, elimintaing a power supply dependency or external buck converter for batteries in systems which use this as the primary processor
Parts:
- removed R16: 0, robot-cortex:R_0402_1005Metric, symbol foc-pcb:Resistor
- added D9: ESD9B3.3ST5G, robot-cortex:D_SOD-923, symbol robot-cortex:ESD9B3.3ST5G
- R13: value 680k -> 365k
- R14: value 130k -> 47k
- U6: now fitted
Connections:
- net GND: now also D9.1 (A1)
- net VBAT: now also D9.2 (A2); no longer C11.1, C12.1, D8.2 (A2), U6.1 (VIN), U6.3 (EN)
- new net 7V0: C11.1, C12.1, D8.2 (A2), U6.1 (VIN), U6.3 (EN)
Changed lines of the file:
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@@
   (junction (at 272.415 231.14) (diameter 0) (color 0 0 0 0)
   )
+  (junction (at 109.855 273.685) (diameter 0) (color 0 0 0 0)
+  )
   (junction (at 206.375 147.955) (diameter 0) (color 0 0 0 0)
   )
@@
     (stroke (width 0) (type default))
   )
+  (wire (pts (xy 104.14 273.685) (xy 109.855 273.685))
+    (stroke (width 0) (type default))
+  )
+  (wire (pts (xy 104.14 265.43) (xy 104.14 266.065))
+    (stroke (width 0) (type default))
+  )
   (wire (pts (xy 160.655 130.175) (xy 160.655 132.715))
     (stroke (width 0) (type default))
@@
     (effects (font (size 1.27 1.27)) (justify left bottom))
   )
-  (label "VUSB" (at 212.725 238.76 180) (fields_autoplaced)
-    (effects (font (size 1.27 1.27)) (justify right bottom))
-  )
   (label "NRST" (at 156.21 67.31 180) (fields_autoplaced)
     (effects (font (size 1.27 1.27)) (justify right bottom))
@@
     (effects (font (size 1.27 1.27)) (justify left bottom))
   )
+  (label "7V0" (at 119.38 194.945 180) (fields_autoplaced)
+    (effects (font (size 1.27 1.27)) (justify right bottom))
+  )
   (label "+5V0" (at 84.455 67.31 0) (fields_autoplaced)
     (effects (font (size 1.27 1.27)) (justify left bottom))
@@
     (effects (font (size 1.27 1.27)) (justify left bottom))
   )
-  (label "VBAT" (at 103.505 194.945 180) (fields_autoplaced)
+  (label "BOOT" (at 271.78 164.465 180) (fields_autoplaced)
     (effects (font (size 1.27 1.27)) (justify right bottom))
   )
-  (label "BOOT" (at 271.78 164.465 180) (fields_autoplaced)
+  (label "VBAT" (at 104.14 265.43 180) (fields_autoplaced)
     (effects (font (size 1.27 1.27)) (justify right bottom))
   )
@@
     (effects (font (size 1.27 1.27)) (justify left bottom))
   )
-  (label "VBAT" (at 80.01 27.94 0) (fields_autoplaced)
-    (effects (font (size 1.27 1.27)) (justify left bottom))
-  )
   (label "LED" (at 209.55 122.555 0) (fields_autoplaced)
     (effects (font (size 1.27 1.27)) (justify left bottom))
@@
     (effects (font (size 1.27 1.27)) (justify left bottom))
   )
+  (label "7V0" (at 82.55 92.075 0) (fields_autoplaced)
+    (effects (font (size 1.27 1.27)) (justify left bottom))
+  )
   (label "+5V0" (at 81.915 31.115 0) (fields_autoplaced)
     (effects (font (size 1.27 1.27)) (justify left bottom))
@@
     (effects (font (size 1.27 1.27)) (justify left bottom))
   )
-  (label "VBAT" (at 82.55 92.075 0) (fields_autoplaced)
-    (effects (font (size 1.27 1.27)) (justify left bottom))
-  )
   (label "+5V0" (at 134.62 196.215 0) (fields_autoplaced)
     (effects (font (size 1.27 1.27)) (justify left bottom))
   )
-  (label "VBAT" (at 109.855 265.43 180) (fields_autoplaced)
-    (effects (font (size 1.27 1.27)) (justify right bottom))
-  )
   (label "+5V0" (at 146.685 196.85 0) (fields_autoplaced)
     (effects (font (size 1.27 1.27)) (justify left bottom))
@@
     (effects (font (size 1.27 1.27)) (justify right bottom))
   )
-  (label "+5V0" (at 275.59 213.36 0) (fields_autoplaced)
+  (label "7V0" (at 275.59 213.36 0) (fields_autoplaced)
     (effects (font (size 1.27 1.27)) (justify left bottom))
   )
@@
     (effects (font (size 1.27 1.27)) (justify right bottom))
   )
-  (label "VBAT" (at 119.38 194.945 180) (fields_autoplaced)
-    (effects (font (size 1.27 1.27)) (justify right bottom))
-  )
   (label "SPI1_SCK" (at 157.48 100.965 180) (fields_autoplaced)
     (effects (font (size 1.27 1.27)) (justify right bottom))
@@
     (effects (font (size 1.27 1.27)) (justify right bottom))
   )
+  (label "7V0" (at 103.505 194.945 180) (fields_autoplaced)
+    (effects (font (size 1.27 1.27)) (justify right bottom))
+  )
   (label "USART2_DE" (at 82.55 80.645 0) (fields_autoplaced)
     (effects (font (size 1.27 1.27)) (justify left bottom))
@@
     (effects (font (size 1.27 1.27)) (justify left bottom))
   )
-  (label "+5V0" (at 220.345 238.76 0) (fields_autoplaced)
+  (label "7V0" (at 109.855 265.43 180) (fields_autoplaced)
+    (effects (font (size 1.27 1.27)) (justify right bottom))
+  )
+  (label "7V0" (at 82.55 64.77 0) (fields_autoplaced)
     (effects (font (size 1.27 1.27)) (justify left bottom))
   )
@@
     (effects (font (size 1.27 1.27)) (justify right bottom))
   )
-  (label "VBAT" (at 82.55 64.77 0) (fields_autoplaced)
-    (effects (font (size 1.27 1.27)) (justify left bottom))
-  )
   (label "D-" (at 315.595 168.91 0) (fields_autoplaced)
     (effects (font (size 1.27 1.27)) (justify left bottom))
@@
     (effects (font (size 1.27 1.27)) (justify left bottom))
   )
+  (label "7V0" (at 80.01 27.94 0) (fields_autoplaced)
+    (effects (font (size 1.27 1.27)) (justify left bottom))
+  )
   (label "VDD_MIXED" (at 238.76 212.725 180) (fields_autoplaced)
     (effects (font (size 1.27 1.27)) (justify right bottom))
@@
   )
   (symbol (lib_id "foc-pcb:SPX3819M5-L-5-0") (at 125.73 200.025 0) (unit 1)
-    (in_bom yes) (on_board yes) (dnp yes)
+    (in_bom yes) (on_board yes) (dnp no)
     (property "Reference" "U6" (at 127 191.77 0)
       (effects (font (size 1.27 1.27)))
@@
       (effects (font (size 1.27 1.27)) (justify left))
     )
-    (property "Value" "130k" (at 276.225 239.395 0)
+    (property "Value" "47k" (at 276.225 239.395 0)
       (effects (font (size 1.27 1.27)))
     )
@@
     )
   )
-  (symbol (lib_id "foc-pcb:Resistor") (at 216.535 238.76 90) (unit 1)
-    (in_bom yes) (on_board yes) (dnp yes)
-    (property "Reference" "R16" (at 217.17 237.49 0)
-      (effects (font (size 1.27 1.27)) (justify left))
-    )
-    (property "Value" "0" (at 219.075 234.95 0)
-      (effects (font (size 1.27 1.27)))
-    )
-    (property "Footprint" "robot-cortex:R_0402_1005Metric" (at 203.835 243.84 0)
-      (effects (font (size 1.27 1.27)) hide)
-    )
-    (property "Datasheet" "~" (at 216.535 238.76 0)
-      (effects (font (size 1.27 1.27)) hide)
-    )
-    (pin "1")
-    (pin "2")
-    (instances
-      (project "robot-cortex"
-        (path "/19e4cb9f-d0a4-4ce0-8aa4-5fe95563dc37"
-          (reference "R16") (unit 1)
-        )
-      )
-      (project "foc-pcb"
-        (path "/2b52ab19-a93e-4439-8602-a1380e4825c0"
-          (reference "R14") (unit 1)
-        )
-      )
-    )
-  )
   (symbol (lib_id "power:+3V3") (at 84.455 34.925 0) (mirror y) (unit 1)
     (in_bom yes) (on_board yes) (dnp no)
@@
       (effects (font (size 1.27 1.27)) (justify left))
     )
-    (property "Value" "680k" (at 276.225 227.965 0)
+    (property "Value" "365k" (at 276.225 227.965 0)
       (effects (font (size 1.27 1.27)))
     )
@@
         )
       )
+    )
+  )
+  (symbol (lib_id "robot-cortex:ESD9B3.3ST5G") (at 104.14 269.875 90) (unit 1)
+    (in_bom yes) (on_board yes) (dnp no)
+    (property "Reference" "D9" (at 101.6 269.875 90)
+      (effects (font (size 1.27 1.27)) (justify right))
+    )
+    (property "Value" "ESD9B3.3ST5G" (at 105.41 276.225 90)
+      (effects (font (size 1.27 1.27)) (justify right) hide)
+    )
+    (property "Footprint" "robot-cortex:D_SOD-923" (at 99.06 267.335 0)
+      (effects (font (size 1.27 1.27)) hide)
+    )
+    (property "Datasheet" "https://www.onsemi.com/pub/Collateral/ESD9B-D.PDF" (at 99.06 267.335 0)
+      (effects (font (size 1.27 1.27)) hide)
+    )
+    (pin "1")
+    (pin "2")
+    (instances
+      (project "robot-cortex"
+        (path "/19e4cb9f-d0a4-4ce0-8aa4-5fe95563dc37"
+          (reference "D9") (unit 1)
+        )
+      )
